Commit message: remove tf_static

File: cow_HW/cow.urdf.xacro (robot description, xacro)
@@ -18,8 +18,10 @@
     <!-- Base footprint -->
     <link name="base_footprint"/>
-    <joint name="base_footprint_to_base_link" type="fixed">
+    <joint name="base_footprint_to_base_link" type="revolute">
         <parent link="base_footprint"/>
         <child link="base_link"/>
         <origin xyz="0 0 0" rpy="0 0 0"/>
+        <axis xyz="0 0 1"/>
+        <limit lower="0" upper="0" effort="0" velocity="0"/>
     </joint>
     <!-- Base link -->
@@ -74,8 +76,10 @@
         </visual>
     </link>
-    <joint name="base_link_to_laser" type="fixed">
+    <joint name="base_link_to_laser" type="revolute">
         <parent link="base_link"/>
         <child link="laser"/>
+        <axis xyz="0 0 1"/>
         <origin xyz="${laser_x} ${laser_y} ${laser_z}" rpy="0 0 0"/>
+        <limit lower="0" upper="0" effort="0" velocity="0"/>
     </joint>
 </robot>

Commit message: change efk and map and urdf

File: cow_HW/cow.urdf.xacro (robot description, xacro)
@@ -18,10 +18,8 @@
     <!-- Base footprint -->
     <link name="base_footprint"/>
-    <joint name="base_footprint_to_base_link" type="revolute">
+    <joint name="base_footprint_to_base_link" type="fixed">
         <parent link="base_footprint"/>
         <child link="base_link"/>
         <origin xyz="0 0 0" rpy="0 0 0"/>
-        <axis xyz="0 0 1"/>
-        <limit lower="0" upper="0" effort="0" velocity="0"/>
     </joint>
     <!-- Base link -->
@@ -76,10 +74,8 @@
         </visual>
     </link>
-    <joint name="base_link_to_laser" type="revolute">
+    <joint name="base_link_to_laser" type="fixed">
         <parent link="base_link"/>
         <child link="laser"/>
-        <axis xyz="0 0 1"/>
         <origin xyz="${laser_x} ${laser_y} ${laser_z}" rpy="0 0 0"/>
-        <limit lower="0" upper="0" effort="0" velocity="0"/>
     </joint>
 </robot>

Commit message: fix urdf and add new urdf

File: cow_HW/cow.urdf.xacro (robot description, xacro)
@@ -15,5 +15,5 @@
     <xacro:property name="laser_x" value="0.145"/>
     <xacro:property name="laser_y" value="0.0"/>
-    <xacro:property name="laser_z" value="0.225"/>
+    <xacro:property name="laser_z" value="0.160"/>
     <!-- Base footprint -->
     <link name="base_footprint"/>
@@ -46,4 +46,9 @@
         </inertial>
     </link>
+    <joint name="base_joint" type="fixed">
+        <parent link="base_link" />
+        <child link="base_footprint" />
+        <origin xyz="0.0 0.0 ${-(wheel_radius+wheel_zoff)}" rpy="0 0 0"/>
+    </joint>
     <!-- Left wheel -->
     <link name="left_wheel"/>
@@ -74,5 +79,5 @@
         </visual>
     </link>
-    <joint name="base_link_to_laser" type="fixed">
+    <joint name="laser_joint" type="fixed">
         <parent link="base_link"/>
         <child link="laser"/>

Commit message: fix launch file

File: cow_HW/cow.urdf.xacro (robot description, xacro)
@@ -18,9 +18,4 @@
     <!-- Base footprint -->
     <link name="base_footprint"/>
-    <joint name="base_footprint_to_base_link" type="fixed">
-        <parent link="base_footprint"/>
-        <child link="base_link"/>
-        <origin xyz="0 0 0" rpy="0 0 0"/>
-    </joint>
     <!-- Base link -->
     <link name="base_link">
@@ -46,7 +41,7 @@
         </inertial>
     </link>
-    <joint name="base_joint" type="fixed">
-        <parent link="base_link" />
-        <child link="base_footprint" />
+    <joint name="base_footprint_to_base_link" type="fixed">
+        <parent link="base_footprint" />
+        <child link="base_link" />
         <origin xyz="0.0 0.0 ${-(wheel_radius+wheel_zoff)}" rpy="0 0 0"/>
     </joint>
@@ -79,5 +74,5 @@
         </visual>
     </link>
-    <joint name="laser_joint" type="fixed">
+    <joint name="base_link_to_laser" type="fixed">
         <parent link="base_link"/>
         <child link="laser"/>

Commit message: laser -> base_sacn

File: cow_HW/cow.urdf.xacro (robot description, xacro)
@@ -63,5 +63,5 @@
     </joint>
     <!-- Laser -->
-    <link name="laser">
+    <link name="base_scan">
         <visual>
             <geometry>
@@ -74,7 +74,7 @@
         </visual>
     </link>
-    <joint name="base_link_to_laser" type="fixed">
+    <joint name="base_link_to_base_scan" type="fixed">
         <parent link="base_link"/>
-        <child link="laser"/>
+        <child link="base_scan"/>
         <origin xyz="${laser_x} ${laser_y} ${laser_z}" rpy="0 0 0"/>
     </joint>
